File: EAGLE/Turnstile.sch (EAGLE design)
At the start: 15 parts

Commit message: OMG, there's a lot on thie board! Added main connector, solar connectors, end cap connector, and new and improved debug connector which is the best thing ever. Good luck Eric!
Parts:
- added CF1: J-HARWIN-M55-60X1242R, J-Harwin-M55-60X1242R-12pin-1.27mm-F-vertical:J-HARWIN-M55-60X1242R
- added J1, J2, J3, J4: Harwin M55-7101242R, J-Harwin-M55-7101242-Solar-card-connector:SOLAR-CARD-CONNECTOR
- added J5: SFM-120-X1-XXX-D, J-Samtec-SFM-120-X1-XXX-D:SFM-120-X1-XXX-D
- added J6: J-SAMTEC-TFM-120-X1-XXX-D-RA, J-Samtec-TFM-120-X1-XXX-D-RA:J-SAMTEC-TFM-120-X1-XXX-D-RA
- added TP1, TP2, TP3, TP4: TEST-POINT-LARGE-SQUARE, oresat-misc:TEST-POINT-LARGE-SQUARE
- PCB1: value ORESAT-CARD-V1.1-3XRF -> ORESAT-CARD-V1.1-END-CARD-3RF-V1.0; device oresat-cards:ORESAT-CARD-V1.1-3XRF -> oresat-cards:ORESAT-CARD-V1.1-END-CARD-3RF-V1.0
Connections:
- new net !SD: J1.!SD, J2.!SD, J3.!SD, J4.!SD, J5.39, J5.40, J6.39, J6.40
- new net CAN1_H: J1.CANH, J2.CANH, J3.CANH, J4.CANH, J5.33, J5.34, J6.33, J6.34
- new net CAN1_L: J1.CANL, J2.CANL, J3.CANL, J4.CANL, J5.35, J5.36, J6.35, J6.36
- new net CAN2_H: J5.17, J5.18, J6.17, J6.18
- new net CAN2_L: J5.19, J5.20, J6.19, J6.20
- new net MAG-POWER: CF1.5, CF1.6, J5.5, J5.6, J6.5, J6.6
- new net MAG-SCL: CF1.3, CF1.4, J5.3, J5.4, J6.3, J6.4
- new net MAG-SDA: CF1.1, CF1.2, J5.1, J5.2, J6.1, J6.2
- new net N$10: J4.AUX, TP4.1
- new net N$7: J1.AUX, TP1.1
- new net N$8: J2.AUX, TP2.1
- new net N$9: J3.AUX, TP3.1
- new net OPD_PWR: J5.15, J5.16, J6.15, J6.16
- new net OPD_SCL: J5.13, J5.14, J6.13, J6.14
- new net OPD_SDA: J5.11, J5.12, J6.11, J6.12
- new net SPARE2: J5.7, J5.8, J6.7, J6.8
- new net TURNSTILE-DEPLOY: J5.10, J5.9, J6.10, J6.9
- new net VBUS: J1.VBUS, J2.VBUS, J3.VBUS, J4.VBUS, J5.21, J5.22, J5.23, J5.24, J5.25, J5.26, J6.21, J6.22, J6.23, J6.24, J6.25, J6.26
- net GND: now also CF1.7, CF1.8, CF1.SHIELDS, J1.GND, J1.SHIELD, J2.GND, J2.SHIELD, J3.GND, J3.SHIELD, J4.GND, J4.SHIELD, J5.27, J5.28, J5.29, J5.30, J5.31, J5.32, J5.37, J5.38, J5.LC1, J5.LC2, J6.27, J6.28, J6.29, J6.30, J6.31, J6.32, J6.37, J6.38
Other:
- note added: "+X"
- note added: "+Y"
- note added: "-X"
- note added: "-Y"
- note added: "1"
- note added: "Main OreSat Card Connector"
- note added: "OreSat Power Domain signals (See power sheet)"
- note added: "OreSat0 +Z End Cap: Solar + Turnstile"
- note added: "TO +Z END CAP"
