File: EAGLE/Mezzanine.sch (EAGLE design)
At the start: 11 parts

Commit message: error checks done
Parts:
- R1, R2, R3: value (none) -> 50
Connections:
- net GND: now also U$13.P$2, U$14.P$2, U$15.P$2, U$16.P$2
Changed lines of the file:
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@@
 <part name="U$10" library="Mini-Circuits-QBA-07+_Phase-shifter" deviceset="QBA-07+" device=""/>
 <part name="U$11" library="Mini-Circuits-QBA-07+_Phase-shifter" deviceset="QBA-07+" device=""/>
-<part name="R1" library="oresat-rcl" deviceset="R-US_" device="0402-A-NOSILK"/>
-<part name="R2" library="oresat-rcl" deviceset="R-US_" device="0402-A-NOSILK"/>
-<part name="R3" library="oresat-rcl" deviceset="R-US_" device="0402-A-NOSILK"/>
+<part name="R1" library="oresat-rcl" deviceset="R-US_" device="0402-A-NOSILK" value="50"/>
+<part name="R2" library="oresat-rcl" deviceset="R-US_" device="0402-A-NOSILK" value="50"/>
+<part name="R3" library="oresat-rcl" deviceset="R-US_" device="0402-A-NOSILK" value="50"/>
 <part name="GND1" library="supply1" library_urn="urn:adsk.eagle:library:371" deviceset="GND" device=""/>
 <part name="GND2" library="supply1" library_urn="urn:adsk.eagle:library:371" deviceset="GND" device=""/>
@@
 <part name="U$15" library="J-HRS-U.FL-R-SMT-1(10)-M-RF" deviceset="U.FL-R-SMA" device=""/>
 <part name="U$16" library="J-HRS-U.FL-R-SMT-1(10)-M-RF" deviceset="U.FL-R-SMA" device=""/>
+<part name="GND7" library="supply1" library_urn="urn:adsk.eagle:library:371" deviceset="GND" device=""/>
+<part name="GND8" library="supply1" library_urn="urn:adsk.eagle:library:371" deviceset="GND" device=""/>
+<part name="GND9" library="supply1" library_urn="urn:adsk.eagle:library:371" deviceset="GND" device=""/>
+<part name="GND10" library="supply1" library_urn="urn:adsk.eagle:library:371" deviceset="GND" device=""/>
 </parts>
 <sheets>
@@
 <attribute name="VALUE" x="234.95" y="83.82" size="1.778" layer="96" rot="MR90"/>
 </instance>
+<instance part="GND7" gate="1" x="223.52" y="147.32" smashed="yes">
+<attribute name="VALUE" x="220.98" y="144.78" size="1.778" layer="96"/>
+</instance>
+<instance part="GND8" gate="1" x="223.52" y="124.46" smashed="yes">
+<attribute name="VALUE" x="220.98" y="121.92" size="1.778" layer="96"/>
+</instance>
+<instance part="GND9" gate="1" x="223.52" y="101.6" smashed="yes">
+<attribute name="VALUE" x="220.98" y="99.06" size="1.778" layer="96"/>
+</instance>
+<instance part="GND10" gate="1" x="223.52" y="78.74" smashed="yes">
+<attribute name="VALUE" x="220.98" y="76.2" size="1.778" layer="96"/>
+</instance>
 </instances>
 <busses>
@@
 <pinref part="U$12" gate="G$1" pin="P$2"/>
 </segment>
+<segment>
+<pinref part="U$13" gate="G$1" pin="P$2"/>
+<pinref part="GND7" gate="1" pin="GND"/>
+<wire x1="223.52" y1="149.86" x2="223.52" y2="152.4" width="0.1524" layer="91"/>
+</segment>
+<segment>
+<pinref part="U$14" gate="G$1" pin="P$2"/>
+<pinref part="GND8" gate="1" pin="GND"/>
+<wire x1="223.52" y1="127" x2="223.52" y2="129.54" width="0.1524" layer="91"/>
+</segment>
+<segment>
+<pinref part="U$15" gate="G$1" pin="P$2"/>
+<pinref part="GND9" gate="1" pin="GND"/>
+<wire x1="223.52" y1="104.14" x2="223.52" y2="106.68" width="0.1524" layer="91"/>
+</segment>
+<segment>
+<pinref part="U$16" gate="G$1" pin="P$2"/>
+<pinref part="GND10" gate="1" pin="GND"/>
+<wire x1="223.52" y1="81.28" x2="223.52" y2="83.82" width="0.1524" layer="91"/>
+</segment>
 </net>
