File: EAGLE/Mezzanine.sch (EAGLE design)
At the start: 11 parts

Commit message: rerouted mezzanine
Parts:
- removed U$12, U$13, U$14, U$15, U$16: U.FL-R-SMA, J-HRS-U.FL-R-SMT-1(10)-M-RF:U.FL-R-SMA
- added U$1, U$2, U$3, U$4, U$5: R107064070, J-Radiall-R107064070-RF:R107064070
Connections:
- net GND: now also U$1.P$2, U$2.P$2, U$3.P$2, U$4.P$2, U$5.P$2; no longer U$12.P$2, U$13.P$2, U$14.P$2, U$15.P$2, U$16.P$2
- net N$1: now also U$1.P$1; no longer U$12.P$1
- net UHF_0: now also U$2.P$1; no longer U$13.P$1
- net UHF_180: now also U$4.P$1; no longer U$15.P$1
- net UHF_270: now also U$5.P$1; no longer U$16.P$1
- net UHF_90: now also U$3.P$1; no longer U$14.P$1
Changed lines of the file:
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@@
 <class number="0" name="default" width="0" drill="0">
+</class>
+<class number="1" name="RF" width="0.38" drill="0.38">
+<clearance class="1" value="1"/>
 </class>
 </classes>
@@
 <part name="GND6" library="supply1" library_urn="urn:adsk.eagle:library:371" deviceset="GND" device=""/>
 <part name="GND14" library="supply1" library_urn="urn:adsk.eagle:library:371" deviceset="GND" device=""/>
-<part name="U$12" library="J-HRS-U.FL-R-SMT-1(10)-M-RF" deviceset="U.FL-R-SMA" device=""/>
-<part name="U$13" library="J-HRS-U.FL-R-SMT-1(10)-M-RF" deviceset="U.FL-R-SMA" device=""/>
-<part name="U$14" library="J-HRS-U.FL-R-SMT-1(10)-M-RF" deviceset="U.FL-R-SMA" device=""/>
-<part name="U$15" library="J-HRS-U.FL-R-SMT-1(10)-M-RF" deviceset="U.FL-R-SMA" device=""/>
-<part name="U$16" library="J-HRS-U.FL-R-SMT-1(10)-M-RF" deviceset="U.FL-R-SMA" device=""/>
 <part name="GND7" library="supply1" library_urn="urn:adsk.eagle:library:371" deviceset="GND" device=""/>
 <part name="GND8" library="supply1" library_urn="urn:adsk.eagle:library:371" deviceset="GND" device=""/>
@@
 <part name="R2" library="oresat-rcl" deviceset="R-US_" device="0805-B-NOSILK" value="50"/>
 <part name="R3" library="oresat-rcl" deviceset="R-US_" device="0805-B-NOSILK" value="50"/>
+<part name="U$1" library="J-Radiall-R107064070-RF" deviceset="R107064070" device=""/>
+<part name="U$2" library="J-Radiall-R107064070-RF" deviceset="R107064070" device=""/>
+<part name="U$3" library="J-Radiall-R107064070-RF" deviceset="R107064070" device=""/>
+<part name="U$4" library="J-Radiall-R107064070-RF" deviceset="R107064070" device=""/>
+<part name="U$5" library="J-Radiall-R107064070-RF" deviceset="R107064070" device=""/>
 </parts>
 <sheets>
@@
 <attribute name="VALUE" x="144.78" y="68.58" size="1.778" layer="96"/>
 </instance>
-<instance part="GND14" gate="1" x="38.1" y="119.38" smashed="yes">
-<attribute name="VALUE" x="35.56" y="116.84" size="1.778" layer="96"/>
-</instance>
-<instance part="U$12" gate="G$1" x="33.02" y="129.54" smashed="yes" rot="R90">
-<attribute name="NAME" x="22.86" y="124.46" size="1.778" layer="95" rot="R90"/>
-<attribute name="VALUE" x="26.67" y="124.46" size="1.778" layer="96" rot="R90"/>
-</instance>
-<instance part="U$13" gate="G$1" x="228.6" y="157.48" smashed="yes" rot="MR90">
-<attribute name="NAME" x="238.76" y="152.4" size="1.778" layer="95" rot="MR90"/>
-<attribute name="VALUE" x="234.95" y="152.4" size="1.778" layer="96" rot="MR90"/>
-</instance>
-<instance part="U$14" gate="G$1" x="228.6" y="134.62" smashed="yes" rot="MR90">
-<attribute name="NAME" x="238.76" y="129.54" size="1.778" layer="95" rot="MR90"/>
-<attribute name="VALUE" x="234.95" y="129.54" size="1.778" layer="96" rot="MR90"/>
-</instance>
-<instance part="U$15" gate="G$1" x="228.6" y="111.76" smashed="yes" rot="MR90">
-<attribute name="NAME" x="238.76" y="106.68" size="1.778" layer="95" rot="MR90"/>
-<attribute name="VALUE" x="234.95" y="106.68" size="1.778" layer="96" rot="MR90"/>
-</instance>
-<instance part="U$16" gate="G$1" x="228.6" y="88.9" smashed="yes" rot="MR90">
-<attribute name="NAME" x="238.76" y="83.82" size="1.778" layer="95" rot="MR90"/>
-<attribute name="VALUE" x="234.95" y="83.82" size="1.778" layer="96" rot="MR90"/>
-</instance>
-<instance part="GND7" gate="1" x="223.52" y="147.32" smashed="yes">
-<attribute name="VALUE" x="220.98" y="144.78" size="1.778" layer="96"/>
-</instance>
-<instance part="GND8" gate="1" x="223.52" y="124.46" smashed="yes">
-<attribute name="VALUE" x="220.98" y="121.92" size="1.778" layer="96"/>
-</instance>
-<instance part="GND9" gate="1" x="223.52" y="101.6" smashed="yes">
-<attribute name="VALUE" x="220.98" y="99.06" size="1.778" layer="96"/>
-</instance>
-<instance part="GND10" gate="1" x="223.52" y="78.74" smashed="yes">
-<attribute name="VALUE" x="220.98" y="76.2" size="1.778" layer="96"/>
+<instance part="GND14" gate="1" x="33.02" y="116.84" smashed="yes">
+<attribute name="VALUE" x="30.48" y="114.3" size="1.778" layer="96"/>
+</instance>
+<instance part="GND7" gate="1" x="228.6" y="144.78" smashed="yes">
+<attribute name="VALUE" x="226.06" y="142.24" size="1.778" layer="96"/>
+</instance>
+<instance part="GND8" gate="1" x="228.6" y="121.92" smashed="yes">
+<attribute name="VALUE" x="226.06" y="119.38" size="1.778" layer="96"/>
+</instance>
+<instance part="GND9" gate="1" x="228.6" y="99.06" smashed="yes">
+<attribute name="VALUE" x="226.06" y="96.52" size="1.778" layer="96"/>
+</instance>
+<instance part="GND10" gate="1" x="228.6" y="76.2" smashed="yes">
+<attribute name="VALUE" x="226.06" y="73.66" size="1.778" layer="96"/>
 </instance>
 <instance part="R1" gate="R" x="68.58" y="114.3" smashed="yes" rot="R90">
@@
 <attribute name="VALUE" x="150.622" y="77.47" size="1.778" layer="96" rot="R90"/>
 </instance>
+<instance part="U$1" gate="G$1" x="33.02" y="129.54" smashed="yes" rot="MR0"/>
+<instance part="U$2" gate="G$1" x="228.6" y="157.48" smashed="yes"/>
+<instance part="U$3" gate="G$1" x="228.6" y="134.62" smashed="yes"/>
+<instance part="U$4" gate="G$1" x="228.6" y="111.76" smashed="yes"/>
+<instance part="U$5" gate="G$1" x="228.6" y="88.9" smashed="yes"/>
 </instances>
 <busses>
 </busses>
 <nets>
-<net name="N$1" class="0">
+<net name="N$1" class="1">
 <segment>
 <pinref part="U$9" gate="G$1" pin="SUM"/>
 <wire x1="38.1" y1="129.54" x2="73.66" y2="129.54" width="0.1524" layer="91"/>
-<pinref part="U$12" gate="G$1" pin="P$1"/>
-</segment>
-</net>
-<net name="N$2" class="0">
+<pinref part="U$1" gate="G$1" pin="P$1"/>
+</segment>
+</net>
+<net name="N$2" class="1">
 <segment>
 <pinref part="U$9" gate="G$1" pin="0"/>
@@
 </segment>
 </net>
-<net name="N$3" class="0">
+<net name="N$3" class="1">
 <segment>
 <pinref part="U$9" gate="G$1" pin="TERM"/>
@@
 <segment>
 <pinref part="GND14" gate="1" pin="GND"/>
-<wire x1="38.1" y1="121.92" x2="38.1" y2="124.46" width="0.1524" layer="91"/>
-<pinref part="U$12" gate="G$1" pin="P$2"/>
-</segment>
-<segment>
-<pinref part="U$13" gate="G$1" pin="P$2"/>
+<wire x1="33.02" y1="119.38" x2="33.02" y2="121.92" width="0.1524" layer="91"/>
+<pinref part="U$1" gate="G$1" pin="P$2"/>
+</segment>
+<segment>
 <pinref part="GND7" gate="1" pin="GND"/>
-<wire x1="223.52" y1="149.86" x2="223.52" y2="152.4" width="0.1524" layer="91"/>
-</segment>
-<segment>
-<pinref part="U$14" gate="G$1" pin="P$2"/>
+<wire x1="228.6" y1="147.32" x2="228.6" y2="149.86" width="0.1524" layer="91"/>
+<pinref part="U$2" gate="G$1" pin="P$2"/>
+</segment>
+<segment>
 <pinref part="GND8" gate="1" pin="GND"/>
-<wire x1="223.52" y1="127" x2="223.52" y2="129.54" width="0.1524" layer="91"/>
-</segment>
-<segment>
-<pinref part="U$15" gate="G$1" pin="P$2"/>
+<wire x1="228.6" y1="124.46" x2="228.6" y2="127" width="0.1524" layer="91"/>
+<pinref part="U$3" gate="G$1" pin="P$2"/>
+</segment>
+<segment>
 <pinref part="GND9" gate="1" pin="GND"/>
-<wire x1="223.52" y1="104.14" x2="223.52" y2="106.68" width="0.1524" layer="91"/>
-</segment>
-<segment>
-<pinref part="U$16" gate="G$1" pin="P$2"/>
+<wire x1="228.6" y1="101.6" x2="228.6" y2="104.14" width="0.1524" layer="91"/>
+<pinref part="U$4" gate="G$1" pin="P$2"/>
+</segment>
+<segment>
 <pinref part="GND10" gate="1" pin="GND"/>
-<wire x1="223.52" y1="81.28" x2="223.52" y2="83.82" width="0.1524" layer="91"/>
-</segment>
-</net>
-<net name="N$4" class="0">
+<wire x1="228.6" y1="78.74" x2="228.6" y2="81.28" width="0.1524" layer="91"/>
+<pinref part="U$5" gate="G$1" pin="P$2"/>
+</segment>
+</net>
+<net name="N$4" class="1">
 <segment>
 <pinref part="U$10" gate="G$1" pin="TERM"/>
@@
 </segment>
 </net>
-<net name="N$5" class="0">
+<net name="N$5" class="1">
 <segment>
 <pinref part="U$11" gate="G$1" pin="SUM"/>
@@
 </segment>
 </net>
-<net name="N$6" class="0">
+<net name="N$6" class="1">
 <segment>
 <pinref part="U$11" gate="G$1" pin="TERM"/>
@@
 </segment>
 </net>
-<net name="UHF_0" class="0">
+<net name="UHF_0" class="1">
 <segment>
 <pinref part="U$10" gate="G$1" pin="0"/>
@@
 <label x="203.2" y="147.32" size="1.778" layer="95"/>
 <wire x1="213.36" y1="147.32" x2="213.36" y2="157.48" width="0.1524" layer="91"/>
-<pinref part="U$13" gate="G$1" pin="P$1"/>
 <wire x1="213.36" y1="157.48" x2="223.52" y2="157.48" width="0.1524" layer="91"/>
-</segment>
-</net>
-<net name="UHF_90" class="0">
+<pinref part="U$2" gate="G$1" pin="P$1"/>
+</segment>
+</net>
+<net name="UHF_90" class="1">
 <segment>
 <pinref part="U$10" gate="G$1" pin="90"/>
@@
 <label x="203.2" y="139.7" size="1.778" layer="95"/>
 <wire x1="213.36" y1="139.7" x2="213.36" y2="134.62" width="0.1524" layer="91"/>
-<pinref part="U$14" gate="G$1" pin="P$1"/>
 <wire x1="213.36" y1="134.62" x2="223.52" y2="134.62" width="0.1524" layer="91"/>
-</segment>
-</net>
-<net name="UHF_270" class="0">
+<pinref part="U$3" gate="G$1" pin="P$1"/>
+</segment>
+</net>
+<net name="UHF_270" class="1">
 <segment>
 <pinref part="U$11" gate="G$1" pin="90"/>
 <label x="203.2" y="88.9" size="1.778" layer="95"/>
 <wire x1="182.88" y1="88.9" x2="223.52" y2="88.9" width="0.1524" layer="91"/>
-<pinref part="U$16" gate="G$1" pin="P$1"/>
-</segment>
-</net>
-<net name="UHF_180" class="0">
+<pinref part="U$5" gate="G$1" pin="P$1"/>
+</segment>
+</net>
+<net name="UHF_180" class="1">
 <segment>
 <pinref part="U$11" gate="G$1" pin="0"/>
@@
 <label x="203.2" y="96.52" size="1.778" layer="95"/>
 <wire x1="213.36" y1="96.52" x2="213.36" y2="111.76" width="0.1524" layer="91"/>
-<pinref part="U$15" gate="G$1" pin="P$1"/>
 <wire x1="213.36" y1="111.76" x2="223.52" y2="111.76" width="0.1524" layer="91"/>
-</segment>
-</net>
+<pinref part="U$4" gate="G$1" pin="P$1"/>
+</segment>
+</net>
