File: EAGLE/Turnstile_ZpC.brd (EAGLE design)
At the start: 99.8 x 94.7 mm, 24 parts, among them J1 Harwin M55-7101242R, J2 Harwin M55-7101242R, J3 Harwin M55-7101242R, J4 Harwin M55-7101242R, J6 J-SAMTEC-TFM-120-X1-XXX-D-RA

Commit message: Corrected Rough draft
Parts:
- moved U$2 7.27 mm to (42.0, 56.0)
- moved U$3 7.27 mm to (57.8, 43.8)
- moved R1 7.07 mm to (65.0, 46.5)
- moved R2 7.07 mm to (60.8, 44.8)
- moved R3 7.07 mm to (39.2, 55.0)
- moved U$1 7.07 mm to (64.0, 50.0)
Routing:
- net N$1: track 55.7 -> 44.0 mm
- net LBAND_90: track 22.9 -> 30.3 mm
- net LBAND_270: track 22.9 -> 30.3 mm
- net LBAND_180: track 22.9 -> 25.2 mm
- net LBAND_0: track 22.9 -> 25.2 mm
- net N$5: track 39.4 -> 41.2 mm
- net N$2: track 9.12 -> 8.57 mm

Commit message: error checks done
Parts:
- R1, R2, R3: value (none) -> 50
