File: EAGLE/Turnstile_ZpC.sch (EAGLE design)
At the start: 24 parts, among them J1 Harwin M55-7101242R, J2 Harwin M55-7101242R, J3 Harwin M55-7101242R, J4 Harwin M55-7101242R, J6 J-SAMTEC-TFM-120-X1-XXX-D-RA

Commit message: error checks done
Parts:
- R1, R2, R3: value (none) -> 50
Changed lines of the file:
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@@
 <parts>
 <part name="FRAME1" library="frames" library_urn="urn:adsk.eagle:library:229" deviceset="FRAME_A_L" device=""/>
-<part name="R1" library="oresat-rcl" deviceset="R-US_" device="0402-A-NOSILK"/>
-<part name="R2" library="oresat-rcl" deviceset="R-US_" device="0402-A-NOSILK"/>
-<part name="R3" library="oresat-rcl" deviceset="R-US_" device="0402-A-NOSILK"/>
+<part name="R1" library="oresat-rcl" deviceset="R-US_" device="0402-A-NOSILK" value="50"/>
+<part name="R2" library="oresat-rcl" deviceset="R-US_" device="0402-A-NOSILK" value="50"/>
+<part name="R3" library="oresat-rcl" deviceset="R-US_" device="0402-A-NOSILK" value="50"/>
 <part name="GND1" library="supply1" library_urn="urn:adsk.eagle:library:371" deviceset="GND" device=""/>
 <part name="GND2" library="supply1" library_urn="urn:adsk.eagle:library:371" deviceset="GND" device=""/>
@@
 </sheet>
 </sheets>
+<errors>
+</errors>
 </schematic>
 </drawing>

Commit message: TestBoard ready for design review and order
Parts:
- R1, R2, R3: value 50 -> (none); device oresat-rcl:R-US_0402-A-NOSILK -> oresat-rcl:R-US_0805-B-NOSILK
Other:
- note added: "MEZZANINE"
- moved on the sheet: CM2, U$2, U$4, U$5, U$6, U$7, U$8
