File: EAGLE/OreSat0_plusZendcard.sch (EAGLE design)
At the start: 11 parts

Commit message: TestBoard ready for design review and order
Parts:
- removed U$10, U$11, U$9: QBA-07+, Mini-Circuits-QBA-07+_Phase-shifter:QBA-07+
- removed U$12, U$13, U$14, U$15, U$16: U.FL-R-SMA, J-HRS-U.FL-R-SMT-1(10)-M-RF:U.FL-R-SMA
- added CF1: J-HARWIN-M55-60X1242R, J-Harwin-M55-60X1242R-12pin-1.27mm-F-vertical:J-HARWIN-M55-60X1242R
- added CM1, CM2: J-MOLEX-SMPM-73300-003X_J-MOLEX-SMPM-73300-003X, J-Molex-SMPM-73300-003X:J-MOLEX-SMPM-73300-003X_J-MOLEX-SMPM-73300-003X
- added J1, J2, J3, J4: Harwin M55-7101242R, J-Harwin-M55-7101242-Solar-card-connector:SOLAR-CARD-CONNECTOR
- added J6: J-SAMTEC-TFM-120-X1-XXX-D-RA, J-Samtec-TFM-120-X1-XXX-D-RA:J-SAMTEC-TFM-120-X1-XXX-D-RA
- added PCB1: ORESAT-CARD-V1.1-END-CARD-3RF-V1.0, oresat-cards:ORESAT-CARD-V1.1-END-CARD-3RF-V1.0
- added TP1, TP2, TP3, TP4: TEST-POINT-LARGE-SQUARE, oresat-misc:TEST-POINT-LARGE-SQUARE
- added U$1, U$2, U$3: QCN-19D+, Mini-Circuits-QCN-19D+_Phase-shifter:QCN-19D+
- added U$4, U$5, U$6, U$7, U$8: U.FL-PR-SMT, J-HRS-U.FL-PR-SMT2.5-1(10)-F-RF:U.FL-PR-SMT
- R1, R2, R3: value 50 -> (none)
Connections:
- new net !SD: J1.!SD, J2.!SD, J3.!SD, J4.!SD, J6.39, J6.40
- new net CAN1_H: J1.CANH, J2.CANH, J3.CANH, J4.CANH, J6.33, J6.34
- new net CAN1_L: J1.CANL, J2.CANL, J3.CANL, J4.CANL, J6.35, J6.36
- new net CAN2_H: J6.17, J6.18
- new net CAN2_L: J6.19, J6.20
- new net LBAND_0: U$3.0
- new net LBAND_180: U$2.0
- new net LBAND_270: U$2.90
- new net LBAND_90: U$3.90
- new net MAG-POWER: CF1.5, CF1.6, J6.5, J6.6
- new net MAG-SCL: CF1.3, CF1.4, J6.3, J6.4
- new net MAG-SDA: CF1.1, CF1.2, J6.1, J6.2
- new net N$10: J4.AUX, TP4.1
- new net N$19: CM2.CENTER, U$4.P$1
- new net N$7: J1.AUX, TP1.1
- new net N$8: J2.AUX, TP2.1
- new net N$9: J3.AUX, TP3.1
- new net OPD_PWR: J6.15, J6.16
- new net OPD_SCL: J6.13, J6.14
- new net OPD_SDA: J6.11, J6.12
- new net SPARE2: J6.7, J6.8
- new net TURNSTILE-DEPLOY: J6.10, J6.9
- new net VBUS: J1.VBUS, J2.VBUS, J3.VBUS, J4.VBUS, J6.21, J6.22, J6.23, J6.24, J6.25, J6.26
- net GND: now also CF1.7, CF1.8, CF1.SHIELDS, CM1.SHIELD, CM1.SHIELD1, CM1.SHIELD2, CM1.SHIELD3, CM2.SHIELD, CM2.SHIELD1, CM2.SHIELD2, CM2.SHIELD3, J1.GND, J1.SHIELD, J2.GND, J2.SHIELD, J3.GND, J3.SHIELD, J4.GND, J4.SHIELD, J6.27, J6.28, J6.29, J6.30, J6.31, J6.32, J6.37, J6.38, U$1.GND, U$2.GND, U$3.GND, U$4.P$2, U$5.P$2, U$6.P$2, U$7.P$2, U$8.P$2; no longer U$10.GND, U$11.GND, U$12.P$2, U$13.P$2, U$14.P$2, U$15.P$2, U$16.P$2, U$9.GND
- net N$1: now also CM1.CENTER, U$1.SUM; no longer U$12.P$1, U$9.SUM
- net N$2: now also U$1.0, U$3.SUM; no longer U$10.SUM, U$9.0
- net N$3: now also U$1.TERM; no longer U$9.TERM
- net N$4: now also U$3.TERM; no longer U$10.TERM
- net N$5: now also U$1.90, U$2.SUM; no longer U$11.SUM, U$9.90
- net N$6: now also U$2.TERM; no longer U$11.TERM
- net UHF_0: now also U$5.P$1; no longer U$10.0, U$13.P$1
- net UHF_180: now also U$7.P$1; no longer U$11.0, U$15.P$1
- net UHF_270: now also U$8.P$1; no longer U$11.90, U$16.P$1
- net UHF_90: now also U$6.P$1; no longer U$10.90, U$14.P$1
Other:
- note added: "+X"
- note added: "+Y"
- note added: "-X"
- note added: "-Y"
- note added: "MEZZANINE"
- note added: "Main OreSat Card Connector"
- note added: "OreSat Power Domain signals (See power sheet)"
- note added: "OreSat0 +Z End Cap: Solar + Turnstile"
- note added: "TO +Z END CAP"
- note removed: "MEZZANINE BOARD FOR UHF FEED SYSTEM"

Commit message: SHIP IT
Parts:
- added R4: HOT, oresat-rcl:R-US_0309/12
- added R5: WARMISH, oresat-rcl:R-US_0309/12
- U$4, U$5, U$6, U$7, U$8: value U.FL-PR-SMT -> R107064070_CONTACT; device J-HRS-U.FL-PR-SMT2.5-1(10)-F-RF:U.FL-PR-SMT -> J-Radiall-R107064070-RF:R107064070_CONTACT
Connections:
- net GND: now also R4.1, R5.1; no longer U$5.P$2, U$6.P$2
- net TURNSTILE-DEPLOY: now also R4.2, R5.2
- net UHF_0: now also U$8.P$1; no longer U$5.P$1
- net UHF_180: now also U$6.P$1; no longer U$7.P$1
- net UHF_270: now also U$5.P$1; no longer U$8.P$1
- net UHF_90: now also U$7.P$1; no longer U$6.P$1

Commit message: error correction
Parts:
- R1, R2, R3: value (none) -> 50
Connections:
- net GND: now also U$5.P$2, U$6.P$2
Changed lines of the file:
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@@
 <part name="GND22" library="supply1" library_urn="urn:adsk.eagle:library:371" deviceset="GND" device=""/>
 <part name="GND7" library="supply1" library_urn="urn:adsk.eagle:library:371" deviceset="GND" device=""/>
-<part name="R1" library="oresat-rcl" deviceset="R-US_" device="0805-B-NOSILK"/>
-<part name="R2" library="oresat-rcl" deviceset="R-US_" device="0805-B-NOSILK"/>
-<part name="R3" library="oresat-rcl" deviceset="R-US_" device="0805-B-NOSILK"/>
+<part name="R1" library="oresat-rcl" deviceset="R-US_" device="0805-B-NOSILK" value="50"/>
+<part name="R2" library="oresat-rcl" deviceset="R-US_" device="0805-B-NOSILK" value="50"/>
+<part name="R3" library="oresat-rcl" deviceset="R-US_" device="0805-B-NOSILK" value="50"/>
 <part name="R4" library="oresat-rcl" deviceset="R-US_" device="0309/12" value="HOT"/>
 <part name="R5" library="oresat-rcl" deviceset="R-US_" device="0309/12" value="WARMISH"/>
@@
 <instance part="U$7" gate="G$1" x="148.59" y="83.82" smashed="yes"/>
 <instance part="U$8" gate="G$1" x="148.59" y="54.61" smashed="yes"/>
-<instance part="GND8" gate="1" x="151.13" y="128.27" smashed="yes">
-<attribute name="VALUE" x="148.59" y="125.73" size="1.778" layer="96"/>
-</instance>
-<instance part="GND9" gate="1" x="151.13" y="100.33" smashed="yes">
-<attribute name="VALUE" x="148.59" y="97.79" size="1.778" layer="96"/>
-</instance>
-<instance part="GND10" gate="1" x="151.13" y="71.12" smashed="yes">
-<attribute name="VALUE" x="148.59" y="68.58" size="1.778" layer="96"/>
-</instance>
-<instance part="GND11" gate="1" x="151.13" y="41.91" smashed="yes">
-<attribute name="VALUE" x="148.59" y="39.37" size="1.778" layer="96"/>
+<instance part="GND8" gate="1" x="151.13" y="125.73" smashed="yes">
+<attribute name="VALUE" x="148.59" y="123.19" size="1.778" layer="96"/>
+</instance>
+<instance part="GND9" gate="1" x="151.13" y="97.79" smashed="yes">
+<attribute name="VALUE" x="148.59" y="95.25" size="1.778" layer="96"/>
+</instance>
+<instance part="GND10" gate="1" x="151.13" y="69.85" smashed="yes">
+<attribute name="VALUE" x="148.59" y="67.31" size="1.778" layer="96"/>
+</instance>
+<instance part="GND11" gate="1" x="151.13" y="40.64" smashed="yes">
+<attribute name="VALUE" x="148.59" y="38.1" size="1.778" layer="96"/>
 </instance>
 </instances>
@@
 <pinref part="U$7" gate="G$1" pin="P$2"/>
 <pinref part="GND10" gate="1" pin="GND"/>
+<wire x1="151.13" y1="72.39" x2="151.13" y2="73.66" width="0.1524" layer="91"/>
 </segment>
 <segment>
 <pinref part="U$8" gate="G$1" pin="P$2"/>
 <pinref part="GND11" gate="1" pin="GND"/>
-</segment>
-</net>
+<wire x1="151.13" y1="43.18" x2="151.13" y2="44.45" width="0.1524" layer="91"/>
+</segment>
+<segment>
+<pinref part="U$5" gate="G$1" pin="P$2"/>
+<pinref part="GND8" gate="1" pin="GND"/>
+<wire x1="151.13" y1="128.27" x2="151.13" y2="129.54" width="0.1524" layer="91"/>
+</segment>
+<segment>
+<pinref part="U$6" gate="G$1" pin="P$2"/>
+<pinref part="GND9" gate="1" pin="GND"/>
+<wire x1="151.13" y1="100.33" x2="151.13" y2="101.6" width="0.1524" layer="91"/>
+</segment>
+</net>

Commit message: Design review cleanup of Eric's perfectly decent board. Added RF class, moved burnwires for maximum OCD placement, cleaned up schematic a little bit.
Other:
- note added: "4x UHF elements (through holes)"
- note added: "L Band Feed System"
- note added: "MEZZANINE PCB"
- note added: "UHF Feed System"
- note added: "UNUSED"
- note removed: "MEZZANINE"
- note removed: "OreSat Power Domain signals (See power sheet)"
Changed lines of the file:
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@@
 <?xml version="1.0" encoding="utf-8"?>
 <!DOCTYPE eagle SYSTEM "eagle.dtd">
-<eagle version="9.6.2">
+<eagle version="9.6.1">
 <drawing>
 <settings>
@@
 <class number="0" name="default" width="0" drill="0">
 </class>
+<class number="1" name="RF" width="0" drill="0">
+<clearance class="1" value="1"/>
+</class>
+<class number="2" name="New Class" width="0" drill="0">
+</class>
 </classes>
 <parts>
@@
 <text x="10.16" y="81.28" size="2.54" layer="97" rot="R90">Main OreSat Card Connector</text>
 <wire x1="110.49" y1="129.54" x2="113.03" y2="129.54" width="0.1524" layer="97"/>
-<wire x1="113.03" y1="129.54" x2="113.03" y2="111.76" width="0.1524" layer="97"/>
-<wire x1="113.03" y1="111.76" x2="110.49" y2="111.76" width="0.1524" layer="97"/>
-<text x="115.57" y="118.11" size="1.778" layer="97">OreSat Power Domain signals
-(See power sheet)</text>
+<wire x1="113.03" y1="129.54" x2="113.03" y2="104.14" width="0.1524" layer="97"/>
+<wire x1="113.03" y1="104.14" x2="110.49" y2="104.14" width="0.1524" layer="97"/>
+<text x="114.3" y="119.38" size="1.778" layer="97">UNUSED</text>
 <text x="223.52" y="120.65" size="1.778" layer="97">+X</text>
 <text x="196.85" y="120.65" size="1.778" layer="97">+Y</text>
@@
 <wire x1="66.04" y1="128.27" x2="66.04" y2="130.81" width="0.1524" layer="91"/>
 <wire x1="15.24" y1="128.27" x2="66.04" y2="128.27" width="0.1524" layer="91"/>
-<label x="115.57" y="133.35" size="2.54" layer="95" xref="yes"/>
+<label x="68.58" y="130.81" size="2.54" layer="95"/>
 <pinref part="J6" gate="G$1" pin="9"/>
 <pinref part="J6" gate="G$1" pin="10"/>
 <junction x="66.04" y="130.81"/>
-<wire x1="66.04" y1="130.81" x2="111.76" y2="130.81" width="0.1524" layer="91"/>
-<wire x1="111.76" y1="130.81" x2="156.21" y2="130.81" width="0.1524" layer="91"/>
+<wire x1="66.04" y1="130.81" x2="156.21" y2="130.81" width="0.1524" layer="91"/>
 <wire x1="156.21" y1="130.81" x2="156.21" y2="148.59" width="0.1524" layer="91"/>
 <pinref part="R5" gate="R" pin="2"/>
@@
 <wire x1="167.64" y1="143.51" x2="167.64" y2="148.59" width="0.1524" layer="91"/>
 <junction x="167.64" y="148.59"/>
-<wire x1="111.76" y1="130.81" x2="111.76" y2="133.35" width="0.1524" layer="91"/>
-<wire x1="111.76" y1="133.35" x2="115.57" y2="133.35" width="0.1524" layer="91"/>
-<junction x="111.76" y="130.81"/>
 </segment>
 </net>
@@
 <wire x1="15.24" y1="90.17" x2="66.04" y2="90.17" width="0.1524" layer="91"/>
 <wire x1="66.04" y1="87.63" x2="66.04" y2="90.17" width="0.1524" layer="91"/>
-<wire x1="95.25" y1="95.25" x2="66.04" y2="95.25" width="0.1524" layer="91"/>
+<wire x1="128.27" y1="95.25" x2="66.04" y2="95.25" width="0.1524" layer="91"/>
 <wire x1="66.04" y1="90.17" x2="66.04" y2="92.71" width="0.1524" layer="91"/>
 <junction x="66.04" y="90.17"/>
@@
 <wire x1="223.52" y1="107.95" x2="196.85" y2="107.95" width="0.1524" layer="91"/>
 <wire x1="196.85" y1="107.95" x2="168.91" y2="107.95" width="0.1524" layer="91"/>
-<wire x1="168.91" y1="107.95" x2="95.25" y2="107.95" width="0.1524" layer="91"/>
-<wire x1="95.25" y1="107.95" x2="95.25" y2="95.25" width="0.1524" layer="91"/>
+<wire x1="168.91" y1="107.95" x2="128.27" y2="107.95" width="0.1524" layer="91"/>
+<wire x1="128.27" y1="107.95" x2="128.27" y2="95.25" width="0.1524" layer="91"/>
 <pinref part="J1" gate="G$1" pin="VBUS"/>
 <junction x="168.91" y="107.95"/>
@@
 <wire x1="143.51" y1="40.64" x2="143.51" y2="156.21" width="0.1524" layer="94"/>
 <wire x1="143.51" y1="156.21" x2="93.98" y2="156.21" width="0.1524" layer="94"/>
-<text x="99.06" y="144.78" size="3.81" layer="94">MEZZANINE</text>
+<text x="104.14" y="138.43" size="3.81" layer="97">MEZZANINE
+PCB</text>
 <wire x1="191.77" y1="157.48" x2="191.77" y2="161.29" width="0.1524" layer="94"/>
 <wire x1="191.77" y1="161.29" x2="187.96" y2="166.37" width="0.1524" layer="94"/>
@@
 <wire x1="238.76" y1="166.37" x2="234.95" y2="161.29" width="0.1524" layer="94"/>
 <wire x1="234.95" y1="161.29" x2="234.95" y2="166.37" width="0.1524" layer="94"/>
+<text x="193.04" y="26.67" size="5.08" layer="94">UHF Feed System</text>
+<wire x1="171.45" y1="182.88" x2="171.45" y2="146.05" width="0.1524" layer="97"/>
+<wire x1="171.45" y1="146.05" x2="256.54" y2="146.05" width="0.1524" layer="97"/>
+<wire x1="256.54" y1="146.05" x2="256.54" y2="182.88" width="0.1524" layer="97"/>
+<wire x1="256.54" y1="182.88" x2="171.45" y2="182.88" width="0.1524" layer="97"/>
+<text x="199.39" y="175.26" size="2.54" layer="97">4x UHF elements
+(through holes)</text>
 </plain>
 <instances>
@@
 </segment>
 </net>
-<net name="UHF_0" class="0">
+<net name="UHF_0" class="1">
 <segment>
 <label x="234.95" y="154.94" size="1.778" layer="95"/>
@@
 </segment>
 </net>
-<net name="UHF_90" class="0">
+<net name="UHF_90" class="1">
 <segment>
 <label x="219.71" y="154.94" size="1.778" layer="95"/>
@@
 </segment>
 </net>
-<net name="UHF_270" class="0">
+<net name="UHF_270" class="1">
 <segment>
 <label x="191.77" y="154.94" size="1.778" layer="95"/>
@@
 </segment>
 </net>
-<net name="UHF_180" class="0">
+<net name="UHF_180" class="1">
 <segment>
 <label x="205.74" y="154.94" size="1.778" layer="95"/>
@@
 </segment>
 </net>
-<net name="N$12" class="0">
+<net name="N$12" class="1">
 <segment>
 <pinref part="U$4" gate="G$1" pin="P$1"/>
@@
 <wire x1="240.03" y1="135.89" x2="237.49" y2="132.08" width="0.1524" layer="94"/>
 <wire x1="237.49" y1="132.08" x2="237.49" y2="135.89" width="0.1524" layer="94"/>
+<text x="194.31" y="26.67" size="5.08" layer="94">L Band Feed System</text>
+<wire x1="212.09" y1="165.1" x2="212.09" y2="128.27" width="0.1524" layer="97"/>
+<wire x1="212.09" y1="128.27" x2="245.11" y2="128.27" width="0.1524" layer="97"/>
+<wire x1="245.11" y1="128.27" x2="245.11" y2="165.1" width="0.1524" layer="97"/>
+<wire x1="245.11" y1="165.1" x2="212.09" y2="165.1" width="0.1524" layer="97"/>
+<text x="214.63" y="156.21" size="2.54" layer="97">4x UHF elements
+(through holes)</text>
 </plain>
 <instances>
@@
 </busses>
 <nets>
-<net name="N$1" class="0">
+<net name="N$1" class="1">
 <segment>
 <wire x1="43.18" y1="129.54" x2="76.2" y2="129.54" width="0.1524" layer="91"/>
@@
 </segment>
 </net>
-<net name="N$2" class="0">
+<net name="N$2" class="1">
 <segment>
 <wire x1="104.14" y1="129.54" x2="114.3" y2="129.54" width="0.1524" layer="91"/>
@@
 </segment>
 </net>
-<net name="N$5" class="0">
+<net name="N$5" class="1">
 <segment>
 <wire x1="139.7" y1="96.52" x2="139.7" y2="101.6" width="0.1524" layer="91"/>
@@
 </segment>
 </net>
-<net name="LBAND_270" class="0">
+<net name="LBAND_270" class="1">
 <segment>
 <label x="238.76" y="138.43" size="1.778" layer="95" rot="R90"/>
@@
 </segment>
 </net>
-<net name="LBAND_180" class="0">
+<net name="LBAND_180" class="1">
 <segment>
 <label x="232.41" y="138.43" size="1.778" layer="95" rot="R90"/>
@@
 </segment>
 </net>
-<net name="LBAND_90" class="0">
+<net name="LBAND_90" class="1">
 <segment>
 <wire x1="184.15" y1="142.24" x2="201.93" y2="142.24" width="0.1524" layer="91"/>
@@
 </segment>
 </net>
-<net name="LBAND_0" class="0">
+<net name="LBAND_0" class="1">
 <segment>
 <wire x1="184.15" y1="147.32" x2="208.28" y2="147.32" width="0.1524" layer="91"/>

Commit message: Updated some parts to have attributes assigned
Parts:
- removed CM1: J-MOLEX-SMPM-73300-003X_J-MOLEX-SMPM-73300-003X, J-Molex-SMPM-73300-003X:J-MOLEX-SMPM-73300-003X_J-MOLEX-SMPM-73300-003X
- added CM3: J-MOLEX-SMPM-73300-003X, J-Molex-SMPM-73300-003X:J-MOLEX-SMPM-73300-003X
- CM2: value J-MOLEX-SMPM-73300-003X_J-MOLEX-SMPM-73300-003X -> J-MOLEX-SMPM-73300-003X; device J-Molex-SMPM-73300-003X:J-MOLEX-SMPM-73300-003X_J-MOLEX-SMPM-73300-003X -> J-Molex-SMPM-73300-003X:J-MOLEX-SMPM-73300-003X
Connections:
- net GND: now also CM3.SHIELD, CM3.SHIELD1, CM3.SHIELD2, CM3.SHIELD3; no longer CM1.SHIELD, CM1.SHIELD1, CM1.SHIELD2, CM1.SHIELD3
- net N$1: now also CM2.CENTER; no longer CM1.CENTER
- net N$12: now also CM3.CENTER; no longer CM2.CENTER
Changed lines of the file:
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@@
 <?xml version="1.0" encoding="utf-8"?>
 <!DOCTYPE eagle SYSTEM "eagle.dtd">
-<eagle version="9.6.1">
+<eagle version="9.6.2">
 <drawing>
 <settings>
@@
 <part name="GND5" library="supply1" library_urn="urn:adsk.eagle:library:371" deviceset="GND" device=""/>
 <part name="GND6" library="supply1" library_urn="urn:adsk.eagle:library:371" deviceset="GND" device=""/>
-<part name="CM1" library="J-Molex-SMPM-73300-003X" deviceset="J-MOLEX-SMPM-73300-003X_J-MOLEX-SMPM-73300-003X" device=""/>
 <part name="FRAME2" library="frames" library_urn="urn:adsk.eagle:library:229" deviceset="FRAME_A_L" device=""/>
-<part name="CM2" library="J-Molex-SMPM-73300-003X" deviceset="J-MOLEX-SMPM-73300-003X_J-MOLEX-SMPM-73300-003X" device=""/>
 <part name="U$1" library="Mini-Circuits-QCN-19D+_Phase-shifter" deviceset="QCN-19D+" device=""/>
 <part name="U$2" library="Mini-Circuits-QCN-19D+_Phase-shifter" deviceset="QCN-19D+" device=""/>
@@
 <part name="GND10" library="supply1" library_urn="urn:adsk.eagle:library:371" deviceset="GND" device=""/>
 <part name="GND11" library="supply1" library_urn="urn:adsk.eagle:library:371" deviceset="GND" device=""/>
+<part name="CM3" library="J-Molex-SMPM-73300-003X" deviceset="J-MOLEX-SMPM-73300-003X" device=""/>
+<part name="CM2" library="J-Molex-SMPM-73300-003X" deviceset="J-MOLEX-SMPM-73300-003X" device=""/>
 </parts>
 <sheets>
@@
 <attribute name="DRAWING_NAME" x="190.5" y="19.05" size="2.54" layer="94"/>
 </instance>
-<instance part="CM2" gate="G$1" x="29.21" y="101.6" smashed="yes">
-<attribute name="NAME" x="34.29" y="97.79" size="1.27" layer="95"/>
-<attribute name="VALUE" x="34.29" y="95.25" size="1.27" layer="95"/>
-</instance>
-<instance part="GND13" gate="1" x="29.21" y="91.44" smashed="yes">
-<attribute name="VALUE" x="26.67" y="88.9" size="1.778" layer="96"/>
+<instance part="GND13" gate="1" x="30.48" y="91.44" smashed="yes">
+<attribute name="VALUE" x="27.94" y="88.9" size="1.778" layer="96"/>
 </instance>
 <instance part="GND7" gate="1" x="86.36" y="80.01" smashed="yes">
@@
 <attribute name="VALUE" x="148.59" y="38.1" size="1.778" layer="96"/>
 </instance>
+<instance part="CM3" gate="G$1" x="30.48" y="101.6" smashed="yes">
+<attribute name="NAME" x="35.56" y="97.79" size="1.27" layer="95"/>
+<attribute name="VALUE" x="35.56" y="95.25" size="1.27" layer="95"/>
+</instance>
 </instances>
 <busses>
@@
 <net name="GND" class="0">
 <segment>
-<pinref part="CM2" gate="G$1" pin="SHIELD3"/>
-<pinref part="CM2" gate="G$1" pin="SHIELD2"/>
-<wire x1="24.13" y1="96.52" x2="26.67" y2="96.52" width="0.1524" layer="91"/>
-<pinref part="CM2" gate="G$1" pin="SHIELD"/>
-<wire x1="26.67" y1="96.52" x2="29.21" y2="96.52" width="0.1524" layer="91"/>
-<wire x1="29.21" y1="96.52" x2="31.75" y2="96.52" width="0.1524" layer="91"/>
-<wire x1="31.75" y1="96.52" x2="34.29" y2="96.52" width="0.1524" layer="91"/>
-<junction x="31.75" y="96.52"/>
-<pinref part="CM2" gate="G$1" pin="SHIELD1"/>
-<junction x="26.67" y="96.52"/>
+<wire x1="25.4" y1="96.52" x2="27.94" y2="96.52" width="0.1524" layer="91"/>
+<wire x1="27.94" y1="96.52" x2="30.48" y2="96.52" width="0.1524" layer="91"/>
+<wire x1="30.48" y1="96.52" x2="33.02" y2="96.52" width="0.1524" layer="91"/>
+<wire x1="33.02" y1="96.52" x2="35.56" y2="96.52" width="0.1524" layer="91"/>
+<junction x="33.02" y="96.52"/>
+<junction x="27.94" y="96.52"/>
 <pinref part="GND13" gate="1" pin="GND"/>
-<wire x1="29.21" y1="93.98" x2="29.21" y2="96.52" width="0.1524" layer="91"/>
-<junction x="29.21" y="96.52"/>
+<wire x1="30.48" y1="93.98" x2="30.48" y2="96.52" width="0.1524" layer="91"/>
+<junction x="30.48" y="96.52"/>
+<pinref part="CM3" gate="G$1" pin="SHIELD"/>
+<pinref part="CM3" gate="G$1" pin="SHIELD1"/>
+<pinref part="CM3" gate="G$1" pin="SHIELD2"/>
+<pinref part="CM3" gate="G$1" pin="SHIELD3"/>
 </segment>
 <segment>
@@
 <segment>
 <pinref part="U$4" gate="G$1" pin="P$1"/>
-<pinref part="CM2" gate="G$1" pin="CENTER"/>
-<wire x1="83.82" y1="101.6" x2="34.29" y2="101.6" width="0.1524" layer="91"/>
+<wire x1="83.82" y1="101.6" x2="35.56" y2="101.6" width="0.1524" layer="91"/>
+<pinref part="CM3" gate="G$1" pin="CENTER"/>
 </segment>
 </net>
@@
 <attribute name="VALUE" x="144.78" y="68.58" size="1.778" layer="96"/>
 </instance>
-<instance part="CM1" gate="G$1" x="38.1" y="129.54" smashed="yes">
-<attribute name="NAME" x="43.18" y="125.73" size="1.27" layer="95"/>
-<attribute name="VALUE" x="43.18" y="123.19" size="1.27" layer="95"/>
-</instance>
 <instance part="U$1" gate="G$1" x="88.9" y="127" smashed="yes">
 <attribute name="NAME" x="81.28" y="134.62" size="1.778" layer="95"/>
@@
 <attribute name="NAME" x="145.8214" y="77.47" size="1.778" layer="95" rot="R90"/>
 <attribute name="VALUE" x="150.622" y="77.47" size="1.778" layer="96" rot="R90"/>
+</instance>
+<instance part="CM2" gate="G$1" x="38.1" y="129.54" smashed="yes">
+<attribute name="NAME" x="43.18" y="125.73" size="1.27" layer="95"/>
+<attribute name="VALUE" x="43.18" y="123.19" size="1.27" layer="95"/>
 </instance>
 </instances>
@@
 <segment>
 <wire x1="43.18" y1="129.54" x2="76.2" y2="129.54" width="0.1524" layer="91"/>
-<pinref part="CM1" gate="G$1" pin="CENTER"/>
 <pinref part="U$1" gate="G$1" pin="SUM"/>
+<pinref part="CM2" gate="G$1" pin="CENTER"/>
 </segment>
 </net>
@@
 </segment>
 <segment>
-<pinref part="CM1" gate="G$1" pin="SHIELD3"/>
-<pinref part="CM1" gate="G$1" pin="SHIELD2"/>
 <wire x1="33.02" y1="124.46" x2="35.56" y2="124.46" width="0.1524" layer="91"/>
-<pinref part="CM1" gate="G$1" pin="SHIELD"/>
 <wire x1="35.56" y1="124.46" x2="38.1" y2="124.46" width="0.1524" layer="91"/>
 <wire x1="38.1" y1="124.46" x2="40.64" y2="124.46" width="0.1524" layer="91"/>
 <wire x1="40.64" y1="124.46" x2="43.18" y2="124.46" width="0.1524" layer="91"/>
 <junction x="40.64" y="124.46"/>
-<pinref part="CM1" gate="G$1" pin="SHIELD1"/>
 <junction x="35.56" y="124.46"/>
 <pinref part="GND14" gate="1" pin="GND"/>
 <wire x1="38.1" y1="121.92" x2="38.1" y2="124.46" width="0.1524" layer="91"/>
 <junction x="38.1" y="124.46"/>
-</segment>
-<segment>
+<pinref part="CM2" gate="G$1" pin="SHIELD"/>
+<pinref part="CM2" gate="G$1" pin="SHIELD1"/>
+<pinref part="CM2" gate="G$1" pin="SHIELD2"/>
+<pinref part="CM2" gate="G$1" pin="SHIELD3"/>
+</segment>
+<segment>
