File: EAGLE/OreSat0_plusZendcard.sch (EAGLE design)
At the start: 26 parts, among them J1 Harwin M55-7101242R, J2 Harwin M55-7101242R, J3 Harwin M55-7101242R, J4 Harwin M55-7101242R, J6 J-SAMTEC-TFM-120-X1-XXX-D-RA

Commit message: +Z end card new outline and fasteners
Parts:
- added U$10, U$11, U$12, U$9: MCMASTER-94100A150, HW-mcmaster-94100A150-M2-threaded-insert:MCMASTER-94100A150
- PCB1: value ORESAT-CARD-V1.1-END-CARD-3RF-V1.0 -> ORESAT-CARD-V1.3-END-CARD-3RF-V1.0; device oresat-cards:ORESAT-CARD-V1.1-END-CARD-3RF-V1.0 -> oresat-cards:ORESAT-CARD-V1.3-END-CARD-3RF-V1.0
Changed lines of the file:
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@@
 </part>
 <part name="GND15" library="supply1" library_urn="urn:adsk.eagle:library:371" deviceset="GND" device=""/>
-<part name="PCB1" library="oresat-cards" deviceset="ORESAT-CARD-V1.1-END-CARD-3RF-V1.0" device=""/>
 <part name="GND16" library="supply1" library_urn="urn:adsk.eagle:library:371" deviceset="GND" device=""/>
 <part name="TP1" library="oresat-misc" deviceset="TEST-POINT-LARGE-SQUARE" device=""/>
@@
 <part name="CM3" library="J-Molex-SMPM-73300-003X" deviceset="J-MOLEX-SMPM-73300-003X" device=""/>
 <part name="CM2" library="J-Molex-SMPM-73300-003X" deviceset="J-MOLEX-SMPM-73300-003X" device=""/>
+<part name="U$9" library="HW-mcmaster-94100A150-M2-threaded-insert" deviceset="MCMASTER-94100A150" device=""/>
+<part name="U$10" library="HW-mcmaster-94100A150-M2-threaded-insert" deviceset="MCMASTER-94100A150" device=""/>
+<part name="U$11" library="HW-mcmaster-94100A150-M2-threaded-insert" deviceset="MCMASTER-94100A150" device=""/>
+<part name="U$12" library="HW-mcmaster-94100A150-M2-threaded-insert" deviceset="MCMASTER-94100A150" device=""/>
+<part name="PCB1" library="oresat-cards" deviceset="ORESAT-CARD-V1.3-END-CARD-3RF-V1.0" device=""/>
 </parts>
 <sheets>
@@
 <attribute name="VALUE" x="97.79" y="48.26" size="1.778" layer="96" rot="MR0"/>
 </instance>
-<instance part="PCB1" gate="G$1" x="63.5" y="27.94" smashed="yes"/>
 <instance part="GND16" gate="1" x="158.75" y="91.44" smashed="yes" rot="MR0">
 <attribute name="VALUE" x="161.29" y="88.9" size="1.778" layer="96" rot="MR0"/>
@@
 <attribute name="VALUE" x="179.07" y="125.73" size="1.778" layer="96" rot="MR0"/>
 </instance>
+<instance part="U$9" gate="G$1" x="48.26" y="10.16" smashed="yes"/>
+<instance part="U$10" gate="G$1" x="55.88" y="10.16" smashed="yes"/>
+<instance part="U$11" gate="G$1" x="63.5" y="10.16" smashed="yes"/>
+<instance part="U$12" gate="G$1" x="71.12" y="10.16" smashed="yes"/>
+<instance part="PCB1" gate="G$1" x="58.42" y="22.86" smashed="yes"/>
 </instances>
 <busses>
